File: rajkoPad.kicad_pcb (KiCad board)
At the start: 2 copper layers, 48.6 x 62.6 mm, 8 parts, among them J1 scl, J2 gnd, J3 3v3, J4 sda, J5 gnd, J6 esp32Left, J7 esp32right, J8 adc

Commit message: Add files via upload
Parts:
- moved J1 21.9 mm to (122.6, 73.5)
- moved J3 9.51 mm to (133.9, 64.1)
- moved J4 7.11 mm to (125.0, 67.4)
- moved J2 6.87 mm to (140.5, 61.1)
Routing:
- net Net-(J1-Pad1): track 30.6 -> 14.8 mm
- net Net-(J2-Pad1): track 16.2 -> 22.9 mm, vias 0 -> 1
- net Net-(J3-Pad1): track 13.6 -> 17.9 mm
- net Net-(J4-Pad1): track 12.2 -> 16.0 mm
Changed lines of the file:
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@@
     (thickness 1.6)
     (drawings 8)
-    (tracks 19)
+    (tracks 23)
     (zones 0)
     (modules 8)
@@
     (visible_elements FFFFFF7F)
     (pcbplotparams
-      (layerselection 0x01000_80000000)
+      (layerselection 0x00000_00000001)
       (usegerberextensions false)
       (excludeedgelayer true)
@@
   )
   (module Wire_Pads:SolderWirePad_single_SMD_5x10mm (layer B.Cu)
-    (at 140.081 60.452)
+    (at 122.555 73.533)
     (descr "Wire Pad, Square, SMD Pad,  5mm x 10mm,")
     (tags "MesurementPoint Square SMDPad 5mmx10mm ")
@@
   )
   (module Wire_Pads:SolderWirePad_single_SMD_5x10mm (layer B.Cu)
-    (at 133.985 63.373)
+    (at 140.462 61.087)
     (descr "Wire Pad, Square, SMD Pad,  5mm x 10mm,")
     (tags "MesurementPoint Square SMDPad 5mmx10mm ")
@@
   )
   (module Wire_Pads:SolderWirePad_single_SMD_5x10mm (layer B.Cu)
-    (at 125.095 67.818)
+    (at 133.858 64.135)
     (descr "Wire Pad, Square, SMD Pad,  5mm x 10mm,")
     (tags "MesurementPoint Square SMDPad 5mmx10mm ")
@@
   )
   (module Wire_Pads:SolderWirePad_single_SMD_5x10mm (layer B.Cu)
-    (at 122.682 74.168)
+    (at 124.968 67.437)
     (descr "Wire Pad, Square, SMD Pad,  5mm x 10mm,")
     (tags "MesurementPoint Square SMDPad 5mmx10mm ")
@@
   (gr_line (start 162.052 113.792) (end 162.052 57.15) (angle 90) (layer Edge.Cuts) (width 0.15))
   (gr_line (start 119.38 113.792) (end 162.052 113.792) (angle 90) (layer Edge.Cuts) (width 0.15))
-  (segment (start 129.54 83.82) (end 134.366 83.82) (width 1.524) (layer B.Cu) (net 1))
-  (segment (start 140.081 78.105) (end 140.081 60.452) (width 1.524) (layer B.Cu) (net 1))
-  (segment (start 134.366 83.82) (end 140.081 78.105) (width 1.524) (layer B.Cu) (net 1))
-  (segment (start 129.54 76.2) (end 132.207 76.2) (width 1.524) (layer B.Cu) (net 2))
-  (segment (start 133.985 74.422) (end 133.985 63.373) (width 1.524) (layer B.Cu) (net 2))
-  (segment (start 132.207 76.2) (end 133.985 74.422) (width 1.524) (layer B.Cu) (net 2))
-  (segment (start 129.54 78.74) (end 128.143 78.74) (width 1.524) (layer B.Cu) (net 3))
-  (segment (start 126.746 77.343) (end 126.746 69.469) (width 1.524) (layer B.Cu) (net 3))
-  (segment (start 128.143 78.74) (end 126.746 77.343) (width 1.524) (layer B.Cu) (net 3))
-  (segment (start 126.746 69.469) (end 125.095 67.818) (width 1.524) (layer B.Cu) (net 3))
-  (segment (start 129.54 81.28) (end 125.73 81.28) (width 1.524) (layer B.Cu) (net 4))
-  (segment (start 122.682 78.232) (end 122.682 74.168) (width 1.524) (layer B.Cu) (net 4))
-  (segment (start 125.73 81.28) (end 122.682 78.232) (width 1.524) (layer B.Cu) (net 4))
+  (segment (start 129.54 83.82) (end 126.746 83.82) (width 1.524) (layer B.Cu) (net 1) (status 400000))
+  (segment (start 122.555 79.629) (end 122.555 73.533) (width 1.524) (layer B.Cu) (net 1) (status 800000))
+  (segment (start 126.746 83.82) (end 122.555 79.629) (width 1.524) (layer B.Cu) (net 1))
+  (segment (start 129.54 76.2) (end 130.556 76.2) (width 1.524) (layer F.Cu) (net 2) (status 400000))
+  (segment (start 140.462 70.866) (end 140.462 61.087) (width 1.524) (layer B.Cu) (net 2) (status 800000))
+  (segment (start 140.335 70.993) (end 140.462 70.866) (width 1.524) (layer B.Cu) (net 2))
+  (via (at 140.335 70.993) (size 0.6) (drill 0.4) (layers F.Cu B.Cu) (net 2))
+  (segment (start 137.414 73.914) (end 140.335 70.993) (width 1.524) (layer F.Cu) (net 2))
+  (segment (start 132.842 73.914) (end 137.414 73.914) (width 1.524) (layer F.Cu) (net 2))
+  (segment (start 130.556 76.2) (end 132.842 73.914) (width 1.524) (layer F.Cu) (net 2))
+  (segment (start 129.54 78.74) (end 132.08 78.74) (width 1.524) (layer B.Cu) (net 3) (status 400000))
+  (segment (start 133.858 76.962) (end 133.858 64.135) (width 1.524) (layer B.Cu) (net 3) (status 800000))
+  (segment (start 132.08 78.74) (end 133.858 76.962) (width 1.524) (layer B.Cu) (net 3))
+  (segment (start 129.54 81.28) (end 129.159 81.28) (width 1.524) (layer B.Cu) (net 4) (status C00000))
+  (segment (start 129.159 81.28) (end 126.746 78.867) (width 1.524) (layer B.Cu) (net 4) (status 400000))
+  (segment (start 126.746 78.867) (end 126.746 69.215) (width 1.524) (layer B.Cu) (net 4) (status 800000))
+  (segment (start 126.746 69.215) (end 124.968 67.437) (width 1.524) (layer B.Cu) (net 4) (status C00000))
   (segment (start 129.54 99.06) (end 132.207 99.06) (width 1.524) (layer B.Cu) (net 5))
   (segment (start 133.985 100.838) (end 133.985 108.204) (width 1.524) (layer B.Cu) (net 5))
